File: Hardware/Haar_Primal.sch (EAGLE design)
At the start: 11 parts, among them J1 CONN_42.54_SCREW, Q1 2N7002, U1 SHT30DFN, U4 DPS368

Commit message: Updated documentation to match standard
Updated docs and readmes, need to add photos of board
Other:
- note added: "ADR 0x44"
- note added: "ADR 0x77"
- moved on the sheet: C1, C3, H1, H2, J1, JP1, Q1, R1, R2, U1, U4
